File: 8bitKeyboardController/8bitKeyboardController.kicad_pcb (KiCad board)
At the start: 2 copper layers, 93.5 x 55 mm, 14 parts

Commit message: Corrections
Correct 3.3V connection for level shifter LV
AGND now connected to GND
Parts:
- renumbered MODE to PS/2
Connections:
- Raspberry_Pi_Pico1 pad 33: unconnected-(Raspberry_Pi_Pico1-AGND-Pad33) -> Net-(C64-Pin_1)
- Raspberry_Pi_Pico1 pad 36: unconnected-(Raspberry_Pi_Pico1-3V3-Pad36) -> Net-(Level-Shifter-1-LV)
- Raspberry_Pi_Pico1 pad 37: Net-(Level-Shifter-1-LV) -> unconnected-(Raspberry_Pi_Pico1-3V3_EN-Pad37)
Routing:
- net Net-(C16-Pin_17): track 118.9 -> 93.5 mm
- net Net-(C64-Pin_4): track 137.6 -> 123.4 mm, vias 1 -> 0
- net Net-(C16-Pin_9): track 75.5 -> 89.2 mm, vias 1 -> 2
- net Net-(C16-Pin_18): track 114.6 -> 102.6 mm
- net Net-(C16-Pin_13): track 54.4 -> 62.9 mm
- net Net-(C16-Pin_7): track 81.0 -> 89.4 mm, vias 1 -> 2
- net Net-(C16-Pin_3): track 83.3 -> 91.2 mm, vias 1 -> 2
- net Net-(C16-Pin_1): track 45.9 -> 53.7 mm, vias 1 -> 0
- net Net-(C16-Pin_11): track 47.7 -> 55.0 mm
- net Net-(C16-Pin_19): track 76.7 -> 83.2 mm
- net Net-(Raspberry_Pi_Pico1-GPIO11): track 44.6 -> 49.8 mm, vias 0 -> 1
- net Net-(C16-Pin_10): track 92.7 -> 88.1 mm
- net Net-(C64-Pin_1): track 221.6 -> 226.0 mm
- net Net-(C16-Pin_12): track 52.8 -> 56.7 mm
- net Net-(C16-Pin_14): track 92.8 -> 90.5 mm, vias 1 -> 0
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